File: Bottom Plate/okey65-bottom-plate.kicad_pcb (KiCad board)
At the start: 2 copper layers, 260.6 x 108.3 mm, 0 parts

Commit message: v 1.0
Other:
- outline, holes or cut-outs redrawn
Changed lines of the file:
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@@
   (general
     (thickness 1.6)
-    (drawings 16)
+    (drawings 17)
     (tracks 0)
     (zones 0)
@@
     (32 B.Adhes user hide)
     (33 F.Adhes user hide)
-    (34 B.Paste user hide)
-    (35 F.Paste user hide)
+    (34 B.Paste user)
+    (35 F.Paste user)
     (36 B.SilkS user)
     (37 F.SilkS user)
@@
     (visible_elements FFFFFF7F)
     (pcbplotparams
-      (layerselection 0x010f0_ffffffff)
-      (usegerberextensions false)
-      (usegerberattributes true)
-      (usegerberadvancedattributes true)
-      (creategerberjobfile true)
+      (layerselection 0x010fc_ffffffff)
+      (usegerberextensions true)
+      (usegerberattributes false)
+      (usegerberadvancedattributes false)
+      (creategerberjobfile false)
       (excludeedgelayer true)
       (linewidth 0.100000)
@@
       (psa4output false)
       (plotreference true)
-      (plotvalue true)
+      (plotvalue false)
       (plotinvisibletext false)
       (padsonsilk false)
@@
     (uvia_drill 0.1)
   )
-  (gr_circle (center 104.812 137.35) (end 105.812 137.35) (layer Edge.Cuts) (width 0.2))
-  (gr_circle (center 20.158573 136.178427) (end 21.158573 136.178427) (layer Edge.Cuts) (width 0.2))
-  (gr_circle (center 188.732558 34.099999) (end 189.732558 34.099999) (layer Edge.Cuts) (width 0.2))
-  (gr_circle (center 273.465427 136.178427) (end 274.465427 136.178427) (layer Edge.Cuts) (width 0.2))
-  (gr_circle (center 188.812 137.35) (end 189.812 137.35) (layer Edge.Cuts) (width 0.2))
-  (gr_circle (center 104.812 34.099999) (end 105.812 34.099999) (layer Edge.Cuts) (width 0.2))
-  (gr_circle (center 273.465427 35.271572) (end 274.465427 35.271572) (layer Edge.Cuts) (width 0.2))
-  (gr_line (start 270.637 31.599999) (end 22.987 31.599999) (layer Edge.Cuts) (width 0.2))
-  (gr_line (start 16.487001 38.099999) (end 16.487001 133.35) (layer Edge.Cuts) (width 0.2))
-  (gr_arc (start 270.637 133.35) (end 270.637 139.85) (angle -90) (layer Edge.Cuts) (width 0.2))
-  (gr_circle (center 20.158573 35.271572) (end 21.158573 35.271572) (layer Edge.Cuts) (width 0.2))
-  (gr_arc (start 270.637 38.099999) (end 277.137 38.099999) (angle -90) (layer Edge.Cuts) (width 0.2))
-  (gr_arc (start 22.987 38.099999) (end 22.987 31.599999) (angle -90) (layer Edge.Cuts) (width 0.2))
-  (gr_line (start 22.987 139.85) (end 270.637 139.85) (layer Edge.Cuts) (width 0.2))
-  (gr_line (start 277.137 133.35) (end 277.137 38.099999) (layer Edge.Cuts) (width 0.2))
-  (gr_arc (start 22.987 133.35) (end 16.487001 133.35) (angle -90) (layer Edge.Cuts) (width 0.2))
+  (gr_arc (start 270.637 38.377) (end 277.137 38.377) (angle -90) (layer Edge.Cuts) (width 0.2))
+  (gr_line (start 270.637 140.127001) (end 22.987 140.127) (layer Edge.Cuts) (width 0.2))
+  (gr_arc (start 22.987 133.627001) (end 16.487001 133.627001) (angle -90) (layer Edge.Cuts) (width 0.2))
+  (gr_circle (center 69.587 60.077) (end 73.787 60.077) (layer Edge.Cuts) (width 0.2))
+  (gr_circle (center 273.465427 136.455428) (end 274.465427 136.455428) (layer Edge.Cuts) (width 0.2))
+  (gr_line (start 16.487001 133.627001) (end 16.487001 38.377) (layer Edge.Cuts) (width 0.2))
+  (gr_circle (center 20.158573 136.455428) (end 21.158573 136.455428) (layer Edge.Cuts) (width 0.2))
+  (gr_circle (center 273.465427 35.548573) (end 274.465427 35.548573) (layer Edge.Cuts) (width 0.2))
+  (gr_arc (start 270.637 133.627001) (end 270.637 140.127001) (angle -90) (layer Edge.Cuts) (width 0.2))
+  (gr_circle (center 188.732558 137.627001) (end 189.732558 137.627001) (layer Edge.Cuts) (width 0.2))
+  (gr_line (start 277.137 38.377) (end 277.137 133.627001) (layer Edge.Cuts) (width 0.2))
+  (gr_circle (center 104.812 34.377) (end 105.812 34.377) (layer Edge.Cuts) (width 0.2))
+  (gr_circle (center 104.812 137.627001) (end 105.812 137.627001) (layer Edge.Cuts) (width 0.2))
+  (gr_circle (center 20.158573 35.548573) (end 21.158573 35.548573) (layer Edge.Cuts) (width 0.2))
+  (gr_circle (center 188.812 34.377) (end 189.812 34.377) (layer Edge.Cuts) (width 0.2))
+  (gr_arc (start 22.987 38.377) (end 22.987 31.877) (angle -90) (layer Edge.Cuts) (width 0.2))
+  (gr_line (start 22.987 31.877) (end 270.637 31.877) (layer Edge.Cuts) (width 0.2))
   (zone (net 0) (net_name "") (layer F.Cu) (hatch edge 0.508)
     (connect_pads (clearance 0.508))
