File: PCB/okey65-pcb.kicad_pcb (KiCad board)
At the start: 2 copper layers, 152 parts, among them J1 USB_C_Receptacle_USB2.0, SW1 SW_Push, U1 ATmega32U4-AU, Y1 16MHz

Commit message: Place all footprints
Parts:
- C1, C2, C3, C4, C5, C6, C7, F1, R1, R2, R3, R4, R6, R7, SW1, U1, Y1: moved to B.Cu
- moved C6 110.6 mm to (77.0, 84.9)
- moved U1 106.2 mm to (81.0, 71.4)
- moved F1 105.6 mm to (58.7, 54.2), turned to 90 degrees
- moved C7 102.5 mm to (67.5, 73.7), turned to 90 degrees
- moved C3 99.7 mm to (69.8, 71.4), turned to 270 degrees
- moved R4 96.2 mm to (86.5, 81.8)
- moved Y1 95.3 mm to (83.3, 57.1), turned to 180 degrees
- moved C5 95.2 mm to (91.3, 67.5), turned to 90 degrees
- moved R3 93.9 mm to (60.3, 45.2), turned to 90 degrees
- moved C4 92.6 mm to (75.4, 57.9)
- moved C2 84.9 mm to (79.4, 57.1), turned to 90 degrees
- moved R6 83.9 mm to (55.6, 38.1), turned to 270 degrees
- moved C1 82.9 mm to (87.3, 57.1), turned to 90 degrees
- moved R2 81.0 mm to (62.7, 45.2), turned to 90 degrees
- moved R1 78.3 mm to (67.5, 57.9), turned to 180 degrees
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
Commit message: Route core circuits
Parts:
- moved D16 3.55 mm to (65.1, 63.5), turned to 0 degrees
- moved C7 3.00 mm to (68.8, 71.0), turned to 270 degrees
- moved C3 2.36 mm to (71.4, 69.7)
Routing:
- net GND: track 0.00 -> 161.7 mm
- net +5V: track 0.00 -> 129.0 mm, vias 0 -> 6
- net Net-(R3-Pad1): track 0.00 -> 38.9 mm
- net Net-(R2-Pad1): track 0.00 -> 37.8 mm
- net VCC: track 0.00 -> 23.1 mm
- net Net-(R1-Pad2): track 0.00 -> 18.2 mm
- net Net-(C1-Pad1): track 0.00 -> 12.2 mm
- net Net-(D3-Pad2): track 0.00 -> 11.9 mm
- net Net-(D17-Pad2): track 0.00 -> 11.9 mm
- net Net-(D30-Pad2): track 0.00 -> 11.9 mm
- net Net-(C2-Pad1): track 0.00 -> 11.6 mm
- net D-: track 0.00 -> 10.8 mm
- net D+: track 0.00 -> 10.2 mm
- net Net-(J1-PadA5): track 0.00 -> 7.20 mm, vias 0 -> 2
- net Net-(D64-Pad2): track 0.00 -> 6.82 mm
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Other:
- net class Default: trace_width 0.25 -> 0.254
- net class Power added: clearance 0.2, trace_width 0.381, via_dia 0.8, via_drill 0.4

Commit message: Routing complete
Parts:
- moved R8 1.59 mm to (154.0, 74.6)
- moved R5 1.59 mm to (39.7, 93.7)
Connections:
- U1 pad 1: Net-(U1-Pad1) -> ROW2
- U1 pad 11: Net-(U1-Pad11) -> COL1
- U1 pad 12: Net-(U1-Pad12) -> COL2
- U1 pad 20: Net-(U1-Pad20) -> ROW0
- U1 pad 21: Net-(U1-Pad21) -> ROW1
- U1 pad 22: Net-(U1-Pad22) -> COL3
- U1 pad 25: Net-(U1-Pad25) -> COL4
- U1 pad 26: Net-(U1-Pad26) -> COL5
- U1 pad 27: Net-(U1-Pad27) -> COL6
- U1 pad 28: Net-(U1-Pad28) -> COL7
- U1 pad 29: Net-(U1-Pad29) -> COL8
- U1 pad 30: Net-(U1-Pad30) -> COL9
- U1 pad 31: Net-(U1-Pad31) -> COL10
- U1 pad 32: Net-(U1-Pad32) -> LED1
- U1 pad 36: Net-(U1-Pad36) -> COL11
- U1 pad 37: Net-(U1-Pad37) -> COL12
- U1 pad 38: Net-(U1-Pad38) -> ROW4
- U1 pad 39: Net-(U1-Pad39) -> ROW3
- U1 pad 40: Net-(U1-Pad40) -> LED0
- U1 pad 41: Net-(U1-Pad41) -> COL0
Routing:
- net ROW0: track 0.00 -> 341.7 mm, vias 0 -> 2
- net ROW4: track 0.00 -> 323.3 mm, vias 0 -> 2
- net ROW1: track 0.00 -> 308.5 mm, vias 0 -> 3
- net ROW3: track 0.00 -> 290.0 mm
- net ROW2: track 0.00 -> 271.2 mm, vias 0 -> 2
- net COL12: track 0.00 -> 268.6 mm
- net COL11: track 0.00 -> 248.2 mm
- net COL10: track 0.00 -> 222.3 mm
- net COL9: track 0.00 -> 202.3 mm
- net COL8: track 0.00 -> 183.0 mm
- net COL7: track 0.00 -> 163.6 mm
- net COL6: track 0.00 -> 144.2 mm
- net COL0: track 0.00 -> 134.9 mm
- net COL5: track 0.00 -> 124.8 mm
- net COL2: track 0.00 -> 120.0 mm, vias 0 -> 3
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
Commit message: PCB complete
Parts:
- moved J1 2.38 mm to (61.9, 31.8)
- moved R6 2.26 mm to (55.6, 35.8)
- moved R7 2.26 mm to (68.3, 35.8)
- moved Y1 0.79 mm to (83.3, 56.3)
- moved C1 0.79 mm to (87.3, 56.4)
- moved C2 0.79 mm to (79.4, 56.4)
Routing:
- net COL3: track 67.7 -> 87.5 mm
- net ROW0: track 341.7 -> 333.6 mm
- net +5V: track 131.7 -> 138.8 mm, vias 6 -> 7
- net GND: track 281.7 -> 286.4 mm, vias 4 -> 5
- net VCC: track 23.1 -> 26.2 mm
- net D-: track 10.8 -> 13.1 mm
- net D+: track 10.2 -> 12.6 mm
- net Net-(C1-Pad1): track 12.2 -> 13.0 mm
- net Net-(C2-Pad1): track 11.6 -> 12.4 mm
- added copper zone on B.Cu, net GND
- added copper zone on F.Cu, net GND
Other:
- board outline added: 255.7 x 103.3 mm
- board text added: "OKey65 rev 1.0"
- board text added: "Powered by QMK"
- board text added: "https://github.com/kiks64/OKey65"

Commit message: Hardware almost complete
Other:
- board size 255.7 x 103.3 mm -> 255.7 x 103.2 mm

Commit message: General improvements - no ground planes
Parts:
- added D68: PRTR5V0U2X, random-keyboard-parts:SOT143B, B.Cu at (61.4, 39.6)
- C7: footprint Capacitor_SMD:C_0805_2012Metric -> Capacitor_SMD:C_1206_3216Metric
- R5, R8: value 80 -> 68
- moved C1 4.31 mm to (83.7, 54.0)
- moved C2 3.15 mm to (81.4, 54.0)
- moved C7 2.69 mm to (69.2, 73.7), turned to 90 degrees
- moved C4 2.38 mm to (77.8, 57.9)
- moved C3 1.55 mm to (71.4, 71.2)
- moved J1 1.52 mm to (61.9, 30.2)
- moved Y1 1.34 mm to (82.6, 57.4)
- moved C5 1.24 mm to (90.0, 67.4)
- moved R6 1.03 mm to (55.6, 34.8)
- moved R7 1.03 mm to (68.3, 34.8)
- moved R2 0.35 mm to (62.4, 45.2)
- moved R3 0.13 mm to (60.5, 45.2)
Routing:
- net GND: track 286.4 -> 272.1 mm, vias 5 -> 23
- net COL9: track 202.3 -> 214.5 mm
- net D+: track 12.6 -> 19.6 mm
- net COL5: track 124.8 -> 130.5 mm
- net +5V: track 138.8 -> 133.9 mm, vias 7 -> 6
- net VCC: track 26.2 -> 28.5 mm
- net D-: track 13.1 -> 15.2 mm
- net Net-(C2-Pad1): track 12.4 -> 11.4 mm
- net ROW0: track 333.6 -> 334.5 mm
- net COL3: track 87.5 -> 86.8 mm
- net Net-(J1-PadA5): track 7.20 -> 7.89 mm
- net Net-(C1-Pad1): track 13.0 -> 13.6 mm
- net Net-(C3-Pad1): track 4.94 -> 4.30 mm
- net Net-(R3-Pad1): track 38.9 -> 38.3 mm
- net Net-(J1-PadB5): track 6.17 -> 6.75 mm
Other:
- board size 255.7 x 103.2 mm -> 255.7 x 104.3 mm
- board text added: "QMK firmware"
- board text removed: "Powered by QMK"

Commit message: v 1.0
Parts:
- added FB1: 60@100MHz, Inductor_SMD:L_1206_3216Metric, B.Cu at (69.6, 30.0)
- R5, R8: value 68 -> 150
- moved SW1 0.79 mm to (70.6, 53.4)
Connections:
- J1 pad S1: GND -> Net-(FB1-Pad2)
Routing:
- net GND: track 272.1 -> 191.3 mm, vias 23 -> 121
- net Net-(FB1-Pad2): track 0.00 -> 19.7 mm, vias 0 -> 3
- added copper zone on B.Cu, net Net-(FB1-Pad2)
- added copper zone on F.Cu, net Net-(FB1-Pad2)
Other:
- board text added: "OKey65"
- board text added: "rev 1.0"
- board text removed: "OKey65 rev 1.0"
